File: speed controller/DRV8323RSRGZT.kicad_sch (KiCad schematic)
At the start: 16 parts, among them U1 DRV8323RSRGZT

Commit message: inital board layout
Parts:
- removed R1: R_Small, symbol Device:R_Small
- removed R4: 10k, symbol Device:R_Small
- added R13, R15: 10k, Resistor_SMD:R_0402_1005Metric, symbol Device:R_Small
- C2, C29: footprint (none) -> Capacitor_SMD:C_0402_1005Metric
- C26, C28, C30: footprint (none) -> Capacitor_SMD:C_0603_1608Metric
- C27: footprint (none) -> Capacitor_SMD:C_1210_3225Metric
- C31: footprint (none) -> Capacitor_SMD:C_1206_3216Metric
- L1: footprint (none) -> Inductor_SMD:DR74
- R5, R6: footprint 54.9k -> Resistor_SMD:R_0402_1005Metric
Connections:
- net +3.3V: now also R13.1
- net Fault: now also R13.2
- net GND: now also R15.2
- net at R5.2, U1.1 (FB): now also R15.1
