File: speed controller/drive.kicad_sch (KiCad schematic)
At the start: 23 parts, among them Q1 IQE022N06LM5CG, Q2 IQE022N06LM5CG, Q3 IQE022N06LM5CG, Q4 IQE022N06LM5CG, Q5 IQE022N06LM5CG, Q6 IQE022N06LM5CG

Commit message: inital board layout
Parts:
- removed C1: 2.2u, symbol Device:C_Small
- removed C5: 100nf, symbol Device:C_Small
- added C33: 2.2u, Capacitor_SMD:C_0603_1608Metric, symbol Device:C_Small
- added C37: 100n, Capacitor_SMD:C_0402_1005Metric, symbol Device:C_Small
- J1, J2, J3: footprint (none) -> TestPoint:TestPoint_THTPad_2.0x2.0mm_Drill1.0mm
- R10, R8, R9: value R_Small -> 1m; footprint (none) -> Resistor_SMD:R_0805_2012Metric
Connections:
- net +3.3V: now also C37.1
- net GND: now also C33.2, C37.2
- net temp: now also C33.1
