File: speed controller/STM32F405RGTx.kicad_sch (KiCad schematic)
At the start: 19 parts, among them U2 STM32F405RGTx, U3 TPS62162DSG, Y1 ECS-80-8-33-JGN-TR3

Commit message: inital board layout
Parts:
- removed C18: 2.2u, symbol Device:C_Small
- added C36: 10p, Capacitor_SMD:C_0402_1005Metric, symbol Device:C_Small
- C15, C23, C3: footprint (none) -> Capacitor_SMD:C_0603_1608Metric
- C16: value 100n -> 2.2u; footprint (none) -> Capacitor_SMD:C_0603_1608Metric
- C17, C19, C20, C21, C22, C24, C34, C4: footprint (none) -> Capacitor_SMD:C_0402_1005Metric
- C35: value 10p -> 100n; footprint (none) -> Capacitor_SMD:C_0402_1005Metric
- L2: footprint (none) -> Inductor_SMD:L_1008_2520Metric
- R7: footprint (none) -> Resistor_SMD:R_0402_1005Metric
- Y1: footprint ECS80833JGNTR3 -> Inductor_SMD:ECS-80-8-33-JGN-TR3
Connections:
- net GND: now also C36.2
- net NRST: now also C35.1; no longer C16.1
- net PH1_OSC_OUT: now also C36.1; no longer C35.1
- net at C15.1, U2.31 (VCAP_1), U2.47 (VCAP_2): now also C16.1

Commit message: trace routing. needs more work on 5v bus. prelem layout complete
Connections:
- net at C16.1, U2.31 (VCAP_1): no longer C15.1, U2.47 (VCAP_2)
- new net: C15.1, U2.47 (VCAP_2)
Other:
- moved on the sheet: C15, C16
Changed lines of the file:
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@@
 	)
 	(junction
-		(at 139.7 166.37)
+		(at 92.71 151.13)
 		(diameter 0)
 		(color 0 0 0 0)
 	)
 	(junction
-		(at 124.46 63.5)
+		(at 139.7 166.37)
 		(diameter 0)
 		(color 0 0 0 0)
 	)
 	(junction
-		(at 92.71 151.13)
+		(at 124.46 63.5)
 		(diameter 0)
 		(color 0 0 0 0)
@@
 	)
 	(junction
-		(at 92.71 137.16)
-		(diameter 0)
-		(color 0 0 0 0)
-	)
-	(junction
-		(at 101.6 137.16)
-		(diameter 0)
-		(color 0 0 0 0)
-	)
-	(junction
 		(at 214.63 111.76)
 		(diameter 0)
@@
 	(wire
 		(pts
-			(xy 101.6 137.16) (xy 92.71 137.16)
+			(xy 83.82 137.16) (xy 104.14 137.16)
 		)
 		(stroke
@@
 	(wire
 		(pts
-			(xy 50.8 31.75) (xy 59.69 31.75)
+			(xy 92.71 147.32) (xy 92.71 151.13)
 		)
 		(stroke
@@
 	(wire
 		(pts
-			(xy 124.46 63.5) (xy 127 63.5)
+			(xy 50.8 31.75) (xy 59.69 31.75)
 		)
 		(stroke
@@
 	(wire
 		(pts
-			(xy 228.6 45.72) (xy 237.49 45.72)
+			(xy 124.46 63.5) (xy 127 63.5)
 		)
 		(stroke
@@
 	(wire
 		(pts
-			(xy 231.14 102.87) (xy 237.49 102.87)
+			(xy 228.6 45.72) (xy 237.49 45.72)
 		)
 		(stroke
@@
 	(wire
 		(pts
-			(xy 83.82 137.16) (xy 83.82 142.24)
+			(xy 231.14 102.87) (xy 237.49 102.87)
 		)
 		(stroke
@@
 	(wire
 		(pts
-			(xy 104.14 137.16) (xy 101.6 137.16)
-		)
-		(stroke
-			(width 0)
-			(type default)
-		)
-	)
-	(wire
-		(pts
 			(xy 127 63.5) (xy 129.54 63.5)
 		)
@@
 	(wire
 		(pts
-			(xy 83.82 147.32) (xy 83.82 151.13)
+			(xy 72.39 62.23) (xy 72.39 63.5)
 		)
 		(stroke
@@
 	(wire
 		(pts
-			(xy 72.39 62.23) (xy 72.39 63.5)
+			(xy 83.82 147.32) (xy 83.82 151.13)
 		)
 		(stroke
@@
 	(wire
 		(pts
-			(xy 92.71 137.16) (xy 92.71 142.24)
+			(xy 121.92 63.5) (xy 124.46 63.5)
 		)
 		(stroke
@@
 	(wire
 		(pts
-			(xy 121.92 63.5) (xy 124.46 63.5)
+			(xy 204.47 63.5) (xy 204.47 66.04)
 		)
 		(stroke
@@
 	(wire
 		(pts
-			(xy 204.47 63.5) (xy 204.47 66.04)
+			(xy 92.71 139.7) (xy 92.71 142.24)
 		)
 		(stroke
@@
 	(wire
 		(pts
-			(xy 104.14 139.7) (xy 101.6 139.7)
+			(xy 92.71 139.7) (xy 104.14 139.7)
 		)
 		(stroke
@@
 	(wire
 		(pts
-			(xy 101.6 139.7) (xy 101.6 137.16)
-		)
-		(stroke
-			(width 0)
-			(type default)
-		)
-	)
-	(wire
-		(pts
 			(xy 214.63 111.76) (xy 231.14 111.76)
 		)
@@
 	(wire
 		(pts
-			(xy 92.71 137.16) (xy 83.82 137.16)
-		)
-		(stroke
-			(width 0)
-			(type default)
-		)
-	)
-	(wire
-		(pts
 			(xy 25.4 36.83) (xy 30.48 36.83)
 		)
@@
 	(wire
 		(pts
-			(xy 92.71 147.32) (xy 92.71 151.13)
-		)
-		(stroke
-			(width 0)
-			(type default)
-		)
-	)
-	(wire
-		(pts
 			(xy 25.4 38.1) (xy 25.4 36.83)
 		)
@@
 		)
 	)
+	(wire
+		(pts
+			(xy 83.82 137.16) (xy 83.82 142.24)
+		)
+		(stroke
+			(width 0)
+			(type default)
+		)
+	)
 	(label "PH1_OSC_OUT"
 		(at 237.49 102.87 0)
@@
 	(symbol
 		(lib_id "Device:C_Small")
-		(at 83.82 144.78 0)
+		(at 92.71 144.78 0)
 		(unit 1)
 		(body_style 1)
@@
 		(fields_autoplaced yes)
 		(property "Reference" "C15"
-			(at 86.36 143.5162 0)
+			(at 95.25 143.5162 0)
 			(show_name no)
 			(do_not_autoplace no)
@@
 		)
 		(property "Value" "2.2u"
-			(at 86.36 146.0562 0)
+			(at 95.25 146.0562 0)
 			(show_name no)
 			(do_not_autoplace no)
@@
 		)
 		(property "Footprint" "Capacitor_SMD:C_0603_1608Metric"
-			(at 83.82 144.78 0)
+			(at 92.71 144.78 0)
 			(hide yes)
 			(show_name no)
@@
 		)
 		(property "Datasheet" "https://www.digikey.com/en/products/detail/samsung-electro-mechanics/CL10A225KO8NNNC/3886698"
-			(at 83.82 144.78 0)
+			(at 92.71 144.78 0)
 			(hide yes)
 			(show_name no)
@@
 		)
 		(property "Description" "Unpolarized capacitor, small symbol"
-			(at 83.82 144.78 0)
+			(at 92.71 144.78 0)
 			(hide yes)
 			(show_name no)
@@
 	(symbol
 		(lib_id "Device:C_Small")
-		(at 92.71 144.78 0)
+		(at 83.82 144.78 0)
 		(unit 1)
 		(body_style 1)
@@
 		(in_pos_files yes)
 		(dnp no)
-		(fields_autoplaced yes)
 		(property "Reference" "C16"
-			(at 95.25 143.5162 0)
+			(at 86.36 143.5162 0)
 			(show_name no)
 			(do_not_autoplace no)
@@
 		)
 		(property "Value" "2.2u"
-			(at 95.25 146.0562 0)
+			(at 86.36 146.0562 0)
 			(show_name no)
 			(do_not_autoplace no)
@@
 		)
 		(property "Footprint" "Capacitor_SMD:C_0603_1608Metric"
-			(at 92.71 144.78 0)
+			(at 83.82 144.78 0)
 			(hide yes)
 			(show_name no)
@@
 		)
 		(property "Datasheet" "https://www.digikey.com/en/products/detail/samsung-electro-mechanics/CL10A225KO8NNNC/3886698"
-			(at 92.71 144.78 0)
+			(at 83.82 144.78 0)
 			(hide yes)
 			(show_name no)
@@
 		)
 		(property "Description" "Unpolarized capacitor, small symbol"
-			(at 92.71 144.78 0)
+			(at 83.82 144.78 0)
 			(hide yes)
 			(show_name no)
